File: STM32F401CCUx/STM32F401CCUx.kicad_pcb (KiCad board)
At the start: 2 copper layers, 5 parts, among them Q1 AO3401A, U3 LM321, U4 STM32F401CCUx, U5 USBLC6-2SC6

Commit message: Update
Parts:
- added R1: 10K, Resistor_SMD:R_1206_3216Metric_Pad1.30x1.75mm_HandSolder, F.Cu at (182.9, 74.9)
- added R10: 62K, Resistor_SMD:R_0402_1005Metric_Pad0.72x0.64mm_HandSolder, F.Cu at (185.6, 83.5)
- added R11: 2K7, Resistor_SMD:R_0402_1005Metric_Pad0.72x0.64mm_HandSolder, F.Cu at (191.6, 80.6)
- added R12: 50, Resistor_SMD:R_0402_1005Metric_Pad0.72x0.64mm_HandSolder, F.Cu at (188.3, 78.6)
- added R13: 1K, Resistor_SMD:R_0402_1005Metric_Pad0.72x0.64mm_HandSolder, F.Cu at (193.3, 73.0)
- added R14: 24K, Resistor_SMD:R_0402_1005Metric_Pad0.72x0.64mm_HandSolder, F.Cu at (182.4, 83.5)
- added R15: 200, Resistor_SMD:R_0402_1005Metric_Pad0.72x0.64mm_HandSolder, F.Cu at (193.3, 71.0)
- added R16: 200, Resistor_SMD:R_0402_1005Metric_Pad0.72x0.64mm_HandSolder, F.Cu at (193.3, 75.0)
- added R17: 1k5, Resistor_SMD:R_0805_2012Metric_Pad1.20x1.40mm_HandSolder, F.Cu at (178.4, 81.7)
- added R18: 1K, Resistor_SMD:R_0805_2012Metric_Pad1.20x1.40mm_HandSolder, F.Cu at (184.3, 78.0)
- added R19: 5K1, Resistor_SMD:R_0402_1005Metric_Pad0.72x0.64mm_HandSolder, F.Cu at (188.9, 82.6)
- added R2: 47k, Resistor_SMD:R_1206_3216Metric_Pad1.30x1.75mm_HandSolder, F.Cu at (173.0, 78.5)
- added R3: 1M, Resistor_SMD:R_0805_2012Metric_Pad1.20x1.40mm_HandSolder, F.Cu at (189.1, 76.1)
- added R4: 1K, Resistor_SMD:R_0805_2012Metric_Pad1.20x1.40mm_HandSolder, F.Cu at (184.3, 81.0)
- added R5: 130k, Resistor_SMD:R_1206_3216Metric_Pad1.30x1.75mm_HandSolder, F.Cu at (182.9, 71.6)
- added R6: 10k, Resistor_SMD:R_1206_3216Metric_Pad1.30x1.75mm_HandSolder, F.Cu at (173.0, 81.8)
- added R7: 6k8, Resistor_SMD:R_1206_3216Metric_Pad1.30x1.75mm_HandSolder, F.Cu at (179.0, 78.5)
- added R8: 47, Resistor_SMD:R_0402_1005Metric_Pad0.72x0.64mm_HandSolder, F.Cu at (191.6, 78.6)
- added R9: 10k, Resistor_SMD:R_0402_1005Metric_Pad0.72x0.64mm_HandSolder, F.Cu at (188.3, 80.6)
- added SW1: SW_SPDT, Button_Switch_SMD:SW_SPDT_PCM12, F.Cu at (175.0, 73.0)
- added U2: EUP3458, Package_TO_SOT_SMD:SOT-23-6_Handsoldering, F.Cu at (188.8, 72.3)

Commit message: PCB
Parts:
- added C1: 10n, Capacitor_SMD:C_0402_1005Metric, F.Cu at (120.0, 122.0)
- added C10: 100n, Capacitor_SMD:C_0603_1608Metric_Pad1.05x0.95mm_HandSolder, F.Cu at (113.5, 109.0)
- added C11: 100n, Capacitor_SMD:C_0603_1608Metric_Pad1.05x0.95mm_HandSolder, F.Cu at (113.4, 107.2)
- added C12: 100n, Capacitor_SMD:C_0603_1608Metric_Pad1.05x0.95mm_HandSolder, F.Cu at (113.4, 105.4)
- added C13: 10n, Capacitor_SMD:C_0402_1005Metric, F.Cu at (112.8, 103.9)
- added C14: 2u2, Capacitor_SMD:CP_Elec_4x5.7, F.Cu at (106.3, 94.5)
- added C15: 10p C335976, Capacitor_SMD:C_0402_1005Metric, F.Cu at (118.4, 103.6)
- added C16: 10p, Capacitor_SMD:C_0402_1005Metric, F.Cu at (126.0, 101.9)
- added C2: 15p, Capacitor_SMD:C_0402_1005Metric, F.Cu at (131.8, 94.2)
- added C3: 15p, Capacitor_SMD:C_0402_1005Metric, F.Cu at (131.8, 91.9)
- added C4: 10n, Capacitor_SMD:C_0402_1005Metric, F.Cu at (120.7, 109.2)
- added C5: 10u, Capacitor_SMD:C_0402_1005Metric, F.Cu at (116.5, 124.0)
- added C6: 10n, Capacitor_SMD:C_0402_1005Metric, F.Cu at (128.5, 91.9)
- added C7: 100n, Capacitor_SMD:C_0603_1608Metric, F.Cu at (131.8, 88.6)
- added C8: 4u7 C116398, Capacitor_SMD:CP_Elec_4x5.3, F.Cu at (108.2, 110.0)
- added C9: 100n, Capacitor_SMD:C_0603_1608Metric_Pad1.05x0.95mm_HandSolder, F.Cu at (113.4, 110.7)
- added D1: B5819W, Diode_SMD:D_SOD-123, F.Cu at (119.7, 127.2)
- added D3: B5819W, Diode_SMD:D_SOD-123, F.Cu at (113.8, 119.8)
- added D4: RED, Diode_SMD:D_0402_1005Metric, F.Cu at (106.2, 115.3)
- added D5: BLUE, Diode_SMD:D_0402_1005Metric, F.Cu at (113.0, 93.2)
- added F1: 250mA, Fuse:Fuseholder_Blade_Mini_Keystone_3568, F.Cu at (126.5, 137.4)
- added FB1: 600 @ 600MHz, Resistor_SMD:R_0805_2012Metric_Pad1.15x1.40mm_HandSolder, F.Cu at (120.0, 124.0)
- added FB2: BLM15AX102SN1D, Resistor_SMD:R_0805_2012Metric_Pad1.15x1.40mm_HandSolder, F.Cu at (129.5, 88.6)
- added J1: Conn_01x04, Connector_PinHeader_2.54mm:PinHeader_1x04_P2.54mm_Horizontal, F.Cu at (99.9, 99.1)
- added J2: Power_Conn, Connector_BarrelJack:BarrelJack_Horizontal, F.Cu at (103.9, 122.2)
- added J3: SWD, Connector_PinHeader_2.54mm:PinHeader_2x05_P2.54mm_Horizontal, F.Cu at (103.6, 89.7)
- added J4: USB_C_Receptacle_USB2.0, Connector_USB:USB_C_Receptacle_HRO_TYPE-C-31-M-12, F.Cu at (94.0, 134.4)
- added L1: 6u8 C395031, Inductor_SMD:L_1206_3216Metric, F.Cu at (114.0, 116.6)
- added L2: 10u C1051, Inductor_SMD:L_1206_3216Metric, F.Cu at (121.7, 106.9)
- added REF**: MountingHole_3.2mm_M3_Pad_Via, MountingHole:MountingHole_3.2mm_M3_Pad_Via, F.Cu at (95.2, 82.0)
- added REF**: MountingHole_3.2mm_M3_Pad_Via, MountingHole:MountingHole_3.2mm_M3_Pad_Via, F.Cu at (131.6, 105.4)
- added REF**: MountingHole_3.2mm_M3_Pad_Via, MountingHole:MountingHole_3.2mm_M3_Pad_Via, F.Cu at (107.7, 135.6)
- added U1: MSM38A2718Z9BM3, MEMS:MEMS38A, F.Cu at (135.0, 87.3)
- added Y1: 25MHz, Crystal:Crystal_SMD_3225-4Pin_3.2x2.5mm_HandSoldering, F.Cu at (122.2, 101.9)
- R1, R2, R5, R6, R7: footprint Resistor_SMD:R_1206_3216Metric_Pad1.30x1.75mm_HandSolder -> Resistor_SMD:R_1206_3216Metric
- R10, R11, R12, R13, R14, R15, R16, R8, R9: footprint Resistor_SMD:R_0402_1005Metric_Pad0.72x0.64mm_HandSolder -> Resistor_SMD:R_0805_2012Metric
- R17, R18, R3, R4: footprint Resistor_SMD:R_0805_2012Metric_Pad1.20x1.40mm_HandSolder -> Resistor_SMD:R_0805_2012Metric
- R19: footprint Resistor_SMD:R_0402_1005Metric_Pad0.72x0.64mm_HandSolder -> Resistor_SMD:R_0402_1005Metric
- moved R19 103.6 mm to (100.8, 137.2), turned to 90 degrees
- moved SW1 91.8 mm to (91.7, 111.5), turned to 270 degrees
- moved R9 90.1 mm to (102.9, 109.1)
- moved R4 88.0 mm to (102.9, 114.3), turned to 270 degrees
- moved U5 84.3 mm to (99.8, 103.9)
- moved U2 83.5 mm to (119.5, 119.0), turned to 180 degrees
- moved R16 80.8 mm to (116.0, 98.3), turned to 90 degrees
- moved R3 80.7 mm to (118.1, 114.6), turned to 270 degrees
- moved R8 80.5 mm to (114.6, 102.1), turned to 180 degrees
- moved R1 79.0 mm to (114.0, 113.6), turned to 180 degrees
- moved R15 77.7 mm to (119.1, 94.0), turned to 90 degrees
- moved Q1 73.6 mm to (124.9, 126.5)
- moved R5 72.7 mm to (123.8, 114.0), turned to 90 degrees
- moved U4 70.2 mm to (107.2, 102.6), turned to 180 degrees
- moved R13 70.2 mm to (126.2, 93.5), turned to 270 degrees
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Routing:
- net +5V: track 0.00 -> 64.7 mm, vias 0 -> 4
- net USB_CONN_D-: track 0.00 -> 45.2 mm, vias 0 -> 3
- net +3V3: track 0.00 -> 41.4 mm, vias 0 -> 18
- net USB_CONN_D+: track 0.00 -> 38.1 mm, vias 0 -> 2
- net GND: track 0.00 -> 24.2 mm, vias 0 -> 3
- net SWO: track 0.00 -> 23.7 mm, vias 0 -> 1
- net SWCLK: track 0.00 -> 23.7 mm, vias 0 -> 1
- net +12V: track 0.00 -> 20.9 mm
- net SWDIO: track 0.00 -> 20.3 mm, vias 0 -> 1
- net BUCK_IN: track 0.00 -> 19.2 mm, vias 0 -> 2
- net NRST: track 0.00 -> 17.0 mm, vias 0 -> 1
- net PWM: track 0.00 -> 14.4 mm, vias 0 -> 3
- net ADC_IN: track 0.00 -> 14.0 mm
- net Net-(C16-Pad1): track 0.00 -> 13.4 mm
- net VDDA: track 0.00 -> 12.4 mm, vias 0 -> 2
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- added copper zone on B.Cu, net +3V3
- added copper zone on F.Cu, net +3V3
- added copper zone on F.Cu, net GND
- added copper zone on F.Cu, net MSM_GND
Other:
- board outline added: 46 x 64.5 mm
- net class Default: clearance 0.2 -> 0.05
- net class Power added: clearance 0.2, trace_width 0.5, via_dia 0.8, via_drill 0.4
- rule trace_clearance: 0.2 -> 0.05
- board text added: "OFF"
- board text added: "ON"

Commit message: Updated PCB
Parts:
- removed the REF** at (95.2, 82.0)
- removed the REF** at (131.6, 105.4)
- removed the REF** at (107.7, 135.6)
- added REF**: MountingHole_3.2mm_M3_Pad_Via, MountingHole:MountingHole_3.2mm_M3_Pad_Via, F.Cu at (94.0, 143.3)
- added REF**: MountingHole_3.2mm_M3_Pad_Via, MountingHole:MountingHole_3.2mm_M3_Pad_Via, F.Cu at (132.0, 143.4)
- added REF**: MountingHole_3.2mm_M3_Pad_Via, MountingHole:MountingHole_3.2mm_M3_Pad_Via, F.Cu at (132.0, 84.0)
- added REF**: MountingHole_3.2mm_M3_Pad_Via, MountingHole:MountingHole_3.2mm_M3_Pad_Via, F.Cu at (94.0, 84.0)
- F1: footprint Fuse:Fuseholder_Blade_Mini_Keystone_3568 -> Fuse_holder:FUSE-TH_L22.6-W9.0
- moved J3 35.7 mm to (128.7, 115.0), turned to 0 degrees
- moved C2 25.2 mm to (107.1, 89.3), turned to 0 degrees
- moved D5 24.9 mm to (106.2, 117.2), turned to 0 degrees
- moved R17 23.7 mm to (102.8, 117.7)
- moved FB2 22.7 mm to (107.1, 85.5)
- moved C3 22.7 mm to (109.4, 88.8)
- moved C7 22.1 mm to (110.0, 85.5)
- moved U1 21.6 mm to (113.6, 84.1)
- moved D2 21.4 mm to (112.7, 89.3)
- moved D1 14.2 mm to (106.2, 122.6), turned to 90 degrees
- moved Q1 13.7 mm to (111.2, 127.1), turned to 270 degrees
- moved C6 11.6 mm to (120.0, 99.8)
- moved J4 11.5 mm to (94.2, 122.9)
- moved R19 11.5 mm to (101.0, 125.7)
- moved J2 11.3 mm to (103.6, 133.5), turned to 90 degrees
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Routing:
- net +3V3: track 41.4 -> 103.0 mm, vias 18 -> 6
- net GND: track 24.2 -> 60.2 mm, vias 3 -> 49
- net CODEC_OUT: track 5.72 -> 38.3 mm
- net LED_STATUS: track 6.24 -> 34.4 mm, vias 0 -> 2
- net +5V: track 64.7 -> 37.2 mm, vias 4 -> 2
- net SWO: track 23.7 -> 49.9 mm
- net SWDIO: track 20.3 -> 43.9 mm
- net SWCLK: track 23.7 -> 47.2 mm
- net NRST: track 17.0 -> 37.4 mm
- net Net-(F1-Pad1): track 11.2 -> 25.6 mm
- net USB_CONN_D-: track 45.2 -> 32.9 mm
- net +12V: track 20.9 -> 8.89 mm
- net USB_CONN_D+: track 38.1 -> 29.4 mm
- net PWM: track 14.4 -> 22.2 mm, vias 3 -> 0
- net PA8: track 9.69 -> 16.4 mm
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- added copper zone on B.Cu, net GND
- added copper zone on B.Cu, net MSM_GND
- removed copper zone on B.Cu, net +3V3
Other:
- board size 46 x 64.5 mm -> 46 x 67.5 mm
- board text added: "12V"
