File: STM32F401CCUx/STM32F401CCUx.sch (KiCad schematic (older format))
At the start: 38 parts

Commit message: Audio Amp and USB Power
Added a pre-amp stage and fixed the USB connections
Parts:
- removed U?: ADC121S051, symbol STM32_Voice:ADC121S051
- added C?: 15p, symbol Device:C_Small
- added D?: B5819W, symbol Device:D_Schottky_Small
- added J?: SWD, symbol Connector_Generic:Conn_02x05_Odd_Even
- added J?: Power_Conn, symbol Connector:Barrel_Jack_Switch
- added J?: USB_C_Receptacle_USB2.0, symbol Connector:USB_C_Receptacle_USB2.0
- added R? (x2): 1K, symbol Device:R_Small
- added R? (x2): 50, symbol Device:R_Small
- added R? (x2): 10K, symbol Device:R_Small
- added R?: 5K1, symbol Device:R_Small
- added U?: LM321, Package_TO_SOT_SMD:SOT-23-5, symbol Amplifier_Operational:LM321
- added U?: USBLC6-2SC6, Package_TO_SOT_SMD:SOT-23-6, symbol Power_Protection:USBLC6-2SC6
- Y?: value 16MHz -> 25MHz
Connections:
- net labels added: +5V, CC, OPAMP_OUT, USB_CONN_D+, USB_CONN_D-
- net labels removed: ADC_CS, ADC_SCLK, ADC_SDATA, ADC_VA, ADC_VIN
- wire segments 114 -> 149
- no-connect marks 25 -> 29
Other:
- note added: "Connectors"
- moved on the sheet: C?, F?, FB?, Q?

Commit message: Updated
Parts:
- added D4: RED, symbol Device:LED_Small
- added J1: Conn_01x04, symbol Connector_Generic:Conn_01x04
- added L2: 10u, symbol Device:L_Small
- added R12: 50, symbol Device:R_Small
- added R16: 200, symbol Device:R_Small
- added R4: 1K, symbol Device:R_Small
- R10: renamed from R?; value 10K -> 62K
- R11: renamed from R?; value 50 -> 2K7
- R14: renamed from R?; value 10K -> 24K
- R15: renamed from R?; value 50 -> 200
- gave numbers to parts that had none: 47
Connections:
- net +3V3: now also U4.1 (VBAT), D4.2 (A), L2.1
- net GND: now also R4.1; no longer R18.1
- net GNDA: now also R18.1
- net ADC_IN: now reaches U4.10 (PA0)
- net ADC_IN: now also U3.4, R16.1
- net PWM: now reaches U4.15 (PA5)
- net PWM: now also J1.1 (Pin_1)
- net PA8: now reaches U4.29 (PA8)
- net PA8: now also J1.2 (Pin_2)
- net PA9: now reaches U4.30 (PA9)
- net PA9: now also J1.3 (Pin_3)
- net PA10: now reaches U4.31 (PA10)
- net PA10: now also J1.4 (Pin_4)
- net VDDA: now reaches U4.9 (VREF+)
- net VDDA: now also L2.2
- net at R13.1, U3.1 (+): now also R12.1; no longer R11.1
- net I2C1_SCL: no longer names the net of U4.42 (PB6)
- net I2C1_SDA: no longer names the net of U4.43 (PB7)
- net OPAMP_OUT: no longer names the net of R15.1
- net OPAMP_OUT: now also R16.2; no longer U3.4
- new net: R11.1, R12.2
- new net: D4.1 (K), R4.2
- no-connect marks 29 -> 25
Other:
- moved on the sheet: C1, C2, C3, C4, C6, C7, D2A, D3, FB2, J2, J3, J4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

Commit message: Update
Parts:
- C8: value 4u7 -> 4u7 C116398
- L1: value 6u8 -> 6u8 C395031; footprint (none) -> Inductor_SMD:L_1206_3216Metric_Pad1.22x1.90mm_HandSolder
- L2: value 10u -> 10u C1051; footprint (none) -> Inductor_SMD:L_1206_3216Metric_Pad1.22x1.90mm_HandSolder
- R1, R2, R5, R6, R7: footprint (none) -> Resistor_SMD:R_1206_3216Metric_Pad1.30x1.75mm_HandSolder
- R10, R11, R12, R13, R14, R15, R16, R17, R18, R3, R4, R8, R9: footprint (none) -> Resistor_SMD:R_0805_2012Metric_Pad1.20x1.40mm_HandSolder
- R19: footprint (none) -> Resistor_SMD:R_0402_1005Metric_Pad0.72x0.64mm_HandSolder
- SW1: footprint (none) -> Button_Switch_SMD:SW_SPDT_PCM12
- U2: footprint (none) -> Package_TO_SOT_SMD:SOT-23-6_Handsoldering
Other:
- note added: "Buck converter"
- note added: "Capacitores próximos ao chip"
- note added: "Chave de BOOT"
- note added: "Circuito de potência"
- note added: "Circuito de proteção"
- note added: "Conectores"
- note added: "Estágio amplificador"
- note added: "MEMs"
- note added: "Microcontrolador"
- note added: "Pinos de saída"
- note added: "Proteção contra ESD no manuseio da entrada USB"
- note removed: "Connectors"
- note removed: "Microcontroller"
- note removed: "Power circuitry"
- moved on the sheet: R9, SW1
Changed lines of the file:
@@
 encoding utf-8
 Sheet 1 1
-Title ""
+Title "Reconhecimentos de voz e comandos de áudio"
 Date ""
 Rev ""
-Comp ""
-Comment1 ""
+Comp "SEMB1"
+Comment1 "Miguel Ravagnani de Carvalho"
 Comment2 ""
 Comment3 ""
@@
 L Switch:SW_SPDT SW1
 U 1 1 606B1396
-P 1650 4350
-F 0 "SW1" H 1650 4635 50  0000 C CNN
-F 1 "SW_SPDT" H 1650 4544 50  0000 C CNN
-F 2 "" H 1650 4350 50  0001 C CNN
-F 3 "~" H 1650 4350 50  0001 C CNN
-	1    1650 4350
+P 1250 5000
+F 0 "SW1" H 1250 5285 50  0000 C CNN
+F 1 "SW_SPDT" H 1250 5194 50  0000 C CNN
+F 2 "Button_Switch_SMD:SW_SPDT_PCM12" H 1250 5000 50  0001 C CNN
+F 3 "~" H 1250 5000 50  0001 C CNN
+	1    1250 5000
 	-1   0    0    -1
 $EndComp
@@
 L Device:R_Small R9
 U 1 1 606B589F
-P 2050 4350
-F 0 "R9" V 1950 4350 50  0000 C CNN
-F 1 "10k" V 2150 4350 50  0000 C CNN
-F 2 "" H 2050 4350 50  0001 C CNN
-F 3 "~" H 2050 4350 50  0001 C CNN
-	1    2050 4350
+P 1650 5000
+F 0 "R9" V 1550 5000 50  0000 C CNN
+F 1 "10k" V 1750 5000 50  0000 C CNN
+F 2 "Resistor_SMD:R_0805_2012Metric_Pad1.20x1.40mm_HandSolder" H 1650 5000 50  0001 C CNN
+F 3 "~" H 1650 5000 50  0001 C CNN
+	1    1650 5000
 	0    -1   1    0
 $EndComp
 Wire Wire Line
-	1950 4350 1850 4350
+	1550 5000 1450 5000
 $Comp
 L power:+3.3V #PWR0104
 U 1 1 606B78FB
-P 1400 4200
-F 0 "#PWR0104" H 1400 4050 50  0001 C CNN
-F 1 "+3.3V" H 1415 4373 50  0000 C CNN
-F 2 "" H 1400 4200 50  0001 C CNN
-F 3 "" H 1400 4200 50  0001 C CNN
-	1    1400 4200
+P 1000 4850
+F 0 "#PWR0104" H 1000 4700 50  0001 C CNN
+F 1 "+3.3V" H 1015 5023 50  0000 C CNN
+F 2 "" H 1000 4850 50  0001 C CNN
+F 3 "" H 1000 4850 50  0001 C CNN
+	1    1000 4850
 	-1   0    0    -1
 $EndComp
 Wire Wire Line
-	1450 4250 1400 4250
-Wire Wire Line
-	1400 4250 1400 4200
+	1050 4900 1000 4900
+Wire Wire Line
+	1000 4900 1000 4850
 $Comp
 L power:GND #PWR0105
 U 1 1 606B8671
-P 1400 4500
-F 0 "#PWR0105" H 1400 4250 50  0001 C CNN
-F 1 "GND" H 1405 4327 50  0000 C CNN
-F 2 "" H 1400 4500 50  0001 C CNN
-F 3 "" H 1400 4500 50  0001 C CNN
-	1    1400 4500
+P 1000 5150
+F 0 "#PWR0105" H 1000 4900 50  0001 C CNN
+F 1 "GND" H 1005 4977 50  0000 C CNN
+F 2 "" H 1000 5150 50  0001 C CNN
+F 3 "" H 1000 5150 50  0001 C CNN
+	1    1000 5150
 	-1   0    0    -1
 $EndComp
 Wire Wire Line
-	1450 4450 1400 4450
-Wire Wire Line
-	1400 4450 1400 4500
-Text GLabel 2150 4350 2    50   Input ~ 0
+	1050 5100 1000 5100
+Wire Wire Line
+	1000 5100 1000 5150
+Text GLabel 1750 5000 2    50   Input ~ 0
 BOOT0
 Text GLabel 4300 4150 0    50   Input ~ 0
@@
 P 900 3350
 F 0 "C8" H 992 3396 50  0000 L CNN
-F 1 "4u7" H 992 3305 50  0000 L CNN
+F 1 "4u7 C116398" H 600 3250 50  0000 L CNN
 F 2 "" H 900 3350 50  0001 C CNN
 F 3 "~" H 900 3350 50  0001 C CNN
@@
 F 0 "R8" H 7550 3900 50  0000 C CNN
 F 1 "47" H 7550 4000 50  0000 C CNN
-F 2 "" H 7650 3950 50  0001 C CNN
+F 2 "Resistor_SMD:R_0805_2012Metric_Pad1.20x1.40mm_HandSolder" H 7650 3950 50  0001 C CNN
 F 3 "~" H 7650 3950 50  0001 C CNN
 	1    7650 3950
@@
 F 0 "R17" H 6950 5350 50  0000 C CNN
 F 1 "1k5" H 6950 5450 50  0000 C CNN
-F 2 "" H 7050 5400 50  0001 C CNN
+F 2 "Resistor_SMD:R_0805_2012Metric_Pad1.20x1.40mm_HandSolder" H 7050 5400 50  0001 C CNN
 F 3 "~" H 7050 5400 50  0001 C CNN
 	1    7050 5400
@@
 F 0 "R3" H 6800 1650 50  0000 C CNN
 F 1 "1M" H 6800 1750 50  0000 C CNN
-F 2 "" H 6900 1700 50  0001 C CNN
+F 2 "Resistor_SMD:R_0805_2012Metric_Pad1.20x1.40mm_HandSolder" H 6900 1700 50  0001 C CNN
 F 3 "~" H 6900 1700 50  0001 C CNN
 	1    6900 1700
@@
 F 0 "R1" H 6800 1250 50  0000 C CNN
 F 1 "10K" H 6800 1350 50  0000 C CNN
-F 2 "" H 6900 1300 50  0001 C CNN
+F 2 "Resistor_SMD:R_1206_3216Metric_Pad1.30x1.75mm_HandSolder" H 6900 1300 50  0001 C CNN
 F 3 "~" H 6900 1300 50  0001 C CNN
 	1    6900 1300
@@
 F 0 "U2" H 4400 2525 50  0000 C CNN
 F 1 "EUP3458" H 4400 2434 50  0000 C CNN
-F 2 "" H 4400 1650 50  0001 C CNN
+F 2 "Package_TO_SOT_SMD:SOT-23-6_Handsoldering" H 4400 1650 50  0001 C CNN
 F 3 "" H 4400 1650 50  0001 C CNN
 	1    4400 1800
@@
 P 5200 1300
 F 0 "L1" V 5385 1300 50  0000 C CNN
-F 1 "6u8" V 5294 1300 50  0000 C CNN
-F 2 "" H 5200 1300 50  0001 C CNN
+F 1 "6u8 C395031" V 5300 1250 50  0000 C CNN
+F 2 "Inductor_SMD:L_1206_3216Metric_Pad1.22x1.90mm_HandSolder" H 5200 1300 50  0001 C CNN
 F 3 "~" H 5200 1300 50  0001 C CNN
 	1    5200 1300
@@
 F 0 "R5" H 5350 1850 50  0000 C CNN
 F 1 "130k" H 5350 1950 50  0000 C CNN
-F 2 "" H 5500 1900 50  0001 C CNN
+F 2 "Resistor_SMD:R_1206_3216Metric_Pad1.30x1.75mm_HandSolder" H 5500 1900 50  0001 C CNN
 F 3 "~" H 5500 1900 50  0001 C CNN
 	1    5500 1900
@@
 F 0 "R2" H 5400 1450 50  0000 C CNN
 F 1 "47k" H 5400 1550 50  0000 C CNN
-F 2 "" H 5500 1500 50  0001 C CNN
+F 2 "Resistor_SMD:R_1206_3216Metric_Pad1.30x1.75mm_HandSolder" H 5500 1500 50  0001 C CNN
 F 3 "~" H 5500 1500 50  0001 C CNN
 	1    5500 1500
@@
 F 0 "R6" H 5650 2050 50  0000 C CNN
 F 1 "10k" H 5650 2150 50  0000 C CNN
-F 2 "" H 5500 2100 50  0001 C CNN
+F 2 "Resistor_SMD:R_1206_3216Metric_Pad1.30x1.75mm_HandSolder" H 5500 2100 50  0001 C CNN
 F 3 "~" H 5500 2100 50  0001 C CNN
 	1    5500 2100
@@
 F 0 "R7" H 5350 2250 50  0000 C CNN
 F 1 "6k8" H 5350 2350 50  0000 C CNN
-F 2 "" H 5500 2300 50  0001 C CNN
+F 2 "Resistor_SMD:R_1206_3216Metric_Pad1.30x1.75mm_HandSolder" H 5500 2300 50  0001 C CNN
 F 3 "~" H 5500 2300 50  0001 C CNN
 	1    5500 2300
@@
 	8600 500  8600 6850
 Text Notes 600  2600 0    100  ~ 0
-Power circuitry
+Circuito de potência
 Text Notes 550  6750 0    100  ~ 0
-Microcontroller
+Microcontrolador
 $Comp
 L power:GND #PWR0118
@@
 F 0 "R18" H 11750 5450 50  0000 C CNN
 F 1 "1K" H 11750 5550 50  0000 C CNN
-F 2 "" H 11850 5500 50  0001 C CNN
+F 2 "Resistor_SMD:R_0805_2012Metric_Pad1.20x1.40mm_HandSolder" H 11850 5500 50  0001 C CNN
 F 3 "~" H 11850 5500 50  0001 C CNN
 	1    11850 5500
@@
 F 0 "R13" V 11400 4950 50  0000 C CNN
 F 1 "1K" V 11200 4950 50  0000 C CNN
-F 2 "" H 11300 4950 50  0001 C CNN
+F 2 "Resistor_SMD:R_0805_2012Metric_Pad1.20x1.40mm_HandSolder" H 11300 4950 50  0001 C CNN
 F 3 "~" H 11300 4950 50  0001 C CNN
 	1    11300 4950
@@
 F 0 "R11" V 11200 4500 50  0000 C CNN
 F 1 "2K7" V 11000 4500 50  0000 C CNN
-F 2 "" H 11100 4500 50  0001 C CNN
+F 2 "Resistor_SMD:R_0805_2012Metric_Pad1.20x1.40mm_HandSolder" H 11100 4500 50  0001 C CNN
 F 3 "~" H 11100 4500 50  0001 C CNN
 	1    11100 4500
@@
 F 0 "R10" V 11000 4500 50  0000 C CNN
 F 1 "62K" V 10800 4500 50  0000 C CNN
-F 2 "" H 10900 4500 50  0001 C CNN
+F 2 "Resistor_SMD:R_0805_2012Metric_Pad1.20x1.40mm_HandSolder" H 10900 4500 50  0001 C CNN
 F 3 "~" H 10900 4500 50  0001 C CNN
 	1    10900 4500
@@
 F 0 "R15" V 12650 5250 50  0000 C CNN
 F 1 "200" V 12450 5250 50  0000 C CNN
-F 2 "" H 12550 5250 50  0001 C CNN
+F 2 "Resistor_SMD:R_0805_2012Metric_Pad1.20x1.40mm_HandSolder" H 12550 5250 50  0001 C CNN
 F 3 "~" H 12550 5250 50  0001 C CNN
 	1    12550 5250
@@
 F 0 "R14" V 12450 5250 50  0000 C CNN
 F 1 "24K" V 12250 5250 50  0000 C CNN
-F 2 "" H 12350 5250 50  0001 C CNN
+F 2 "Resistor_SMD:R_0805_2012Metric_Pad1.20x1.40mm_HandSolder" H 12350 5250 50  0001 C CNN
 F 3 "~" H 12350 5250 50  0001 C CNN
 	1    12350 5250
@@
 	11850 5250 12250 5250
 Text Notes 550  11100 0    100  ~ 0
-Connectors
+Conectores
 $Comp
 L power:+3.3V #PWR0126
@@
 F 0 "R19" H 4650 8050 50  0000 C CNN
 F 1 "5K1" H 4650 8150 50  0000 C CNN
-F 2 "" H 4800 8100 50  0001 C CNN
+F 2 "Resistor_SMD:R_0402_1005Metric_Pad0.72x0.64mm_HandSolder" H 4800 8100 50  0001 C CNN
 F 3 "~" H 4800 8100 50  0001 C CNN
 	1    4800 8100
@@
 F 0 "R4" H 7850 1650 50  0000 C CNN
 F 1 "1K" H 7850 1750 50  0000 C CNN
-F 2 "" H 8000 1700 50  0001 C CNN
+F 2 "Resistor_SMD:R_0805_2012Metric_Pad1.20x1.40mm_HandSolder" H 8000 1700 50  0001 C CNN
 F 3 "~" H 8000 1700 50  0001 C CNN
 	1    8000 1700
@@
 F 0 "R12" V 11400 4500 50  0000 C CNN
 F 1 "50" V 11200 4500 50  0000 C CNN
-F 2 "" H 11300 4500 50  0001 C CNN
+F 2 "Resistor_SMD:R_0805_2012Metric_Pad1.20x1.40mm_HandSolder" H 11300 4500 50  0001 C CNN
 F 3 "~" H 11300 4500 50  0001 C CNN
 	1    11300 4500
@@
 F 0 "R16" V 12850 5250 50  0000 C CNN
 F 1 "200" V 12650 5250 50  0000 C CNN
-F 2 "" H 12750 5250 50  0001 C CNN
+F 2 "Resistor_SMD:R_0805_2012Metric_Pad1.20x1.40mm_HandSolder" H 12750 5250 50  0001 C CNN
 F 3 "~" H 12750 5250 50  0001 C CNN
 	1    12750 5250
@@
 P 7150 2450
 F 0 "L2" V 7335 2450 50  0000 C CNN
-F 1 "10u" V 7244 2450 50  0000 C CNN
-F 2 "" H 7150 2450 50  0001 C CNN
+F 1 "10u C1051" V 7244 2450 50  0000 C CNN
+F 2 "Inductor_SMD:L_1206_3216Metric_Pad1.22x1.90mm_HandSolder" H 7150 2450 50  0001 C CNN
 F 3 "~" H 7150 2450 50  0001 C CNN
 	1    7150 2450
@@
 Wire Wire Line
 	4050 7600 4050 7700
+Text Notes 800  750  0    50   ~ 0
+Circuito de proteção
+Text Notes 3650 750  0    50   ~ 0
+Buck converter
+Text Notes 9750 800  0    50   ~ 0
+MEMs
+Text Notes 10550 3950 0    50   ~ 0
+Estágio amplificador
+Text Notes 900  5550 0    50   ~ 0
+Chave de BOOT
+Text Notes 850  4000 0    50   ~ 0
+Capacitores próximos ao chip
+Text Notes 6200 8900 0    50   ~ 0
+Proteção contra ESD no manuseio da entrada USB
+Text Notes 9650 8500 0    50   ~ 0
+Pinos de saída
 $EndSCHEMATC

Commit message: PCB
Parts:
- C1, C13, C16, C2, C3, C4, C5, C6: footprint (none) -> Capacitor_SMD:C_0402_1005Metric
- C10, C11, C12, C9: footprint (none) -> Capacitor_SMD:C_0603_1608Metric_Pad1.05x0.95mm_HandSolder
- C14: footprint (none) -> Capacitor_SMD:CP_Elec_4x5.7
- C15: value 10p -> 10p C335976; footprint (none) -> Capacitor_SMD:C_0402_1005Metric
- C7: footprint (none) -> Capacitor_SMD:C_0603_1608Metric
- C8: footprint (none) -> Capacitor_SMD:CP_Elec_4x5.3
- D1, D3: footprint (none) -> Diode_SMD:D_SOD-123
- D4, D5: footprint (none) -> Diode_SMD:D_0402_1005Metric
- F1: footprint (none) -> Fuse:Fuseholder_Blade_Mini_Keystone_3568
- FB1, FB2: footprint (none) -> Resistor_SMD:R_0805_2012Metric_Pad1.15x1.40mm_HandSolder
- J1: footprint (none) -> Connector_PinHeader_2.54mm:PinHeader_1x04_P2.54mm_Horizontal
- J2: footprint (none) -> Connector_BarrelJack:BarrelJack_Horizontal
- J3: footprint (none) -> Connector_PinHeader_2.54mm:PinHeader_2x05_P2.54mm_Horizontal
- J4: footprint (none) -> Connector_USB:USB_C_Receptacle_HRO_TYPE-C-31-M-12; symbol Connector:USB_C_Receptacle_USB2.0 -> STM32F401CCUx-rescue:USB_C_Receptacle_USB2.0-Connector
- L1, L2: footprint Inductor_SMD:L_1206_3216Metric_Pad1.22x1.90mm_HandSolder -> Inductor_SMD:L_1206_3216Metric
- R1, R2, R5, R6, R7: footprint Resistor_SMD:R_1206_3216Metric_Pad1.30x1.75mm_HandSolder -> Resistor_SMD:R_1206_3216Metric
- R10, R11, R12, R13, R14, R15, R16, R17, R18, R3, R4, R8, R9: footprint Resistor_SMD:R_0805_2012Metric_Pad1.20x1.40mm_HandSolder -> Resistor_SMD:R_0805_2012Metric
- R19: footprint Resistor_SMD:R_0402_1005Metric_Pad0.72x0.64mm_HandSolder -> Resistor_SMD:R_0402_1005Metric
- U1: footprint (none) -> MEMS:MEMS38A
- U5: symbol Power_Protection:USBLC6-2SC6 -> STM32F401CCUx-rescue:USBLC6-2SC6-Power_Protection
- Y1: footprint (none) -> Crystal:Crystal_SMD_3225-4Pin_3.2x2.5mm_HandSoldering

Commit message: Updated PCB
Parts:
- F1: footprint Fuse:Fuseholder_Blade_Mini_Keystone_3568 -> Fuse_holder:FUSE-TH_L22.6-W9.0
Connections:
- net PA10: now also J1.1 (Pin_1); no longer J1.4 (Pin_4)
- net PA8: now also J1.3 (Pin_3); no longer J1.2 (Pin_2)
- net PA9: now also J1.2 (Pin_2); no longer J1.3 (Pin_3)
- net PWM: now also J1.4 (Pin_4); no longer J1.1 (Pin_1)
Changed lines of the file:
@@
 F 0 "F1" V 925 1350 50  0000 C CNN
 F 1 "250mA" V 1016 1350 50  0000 C CNN
-F 2 "Fuse:Fuseholder_Blade_Mini_Keystone_3568" H 1200 1150 50  0001 L CNN
+F 2 "Fuse_holder:FUSE-TH_L22.6-W9.0" H 1200 1150 50  0001 L CNN
 F 3 "~" H 1150 1350 50  0001 C CNN
 	1    1150 1350
@@
 	1    0    0    -1
 $EndComp
+Text GLabel 9850 8050 0    50   Input ~ 0
+PA8
 Text GLabel 9850 7950 0    50   Input ~ 0
-PA8
-Text GLabel 9850 8050 0    50   Input ~ 0
 PA9
+Text GLabel 9850 7850 0    50   Input ~ 0
+PA10
 Text GLabel 9850 8150 0    50   Input ~ 0
-PA10
-Text GLabel 9850 7850 0    50   Input ~ 0
 PWM
 $Comp
